Commit message: center the camera meshes, add projection frame

File: urdf/macros/zivid_one_plus_camera.xacro (robot description, xacro)
@@ -17,6 +17,7 @@
         <link name="${prefix}base_link">
             <!-- Visuals -->
+            <!-- vendor stl was centred on projection frame -->
             <visual>
-                <origin xyz="-0.0030 -0.0758 0.0445" rpy="${0.5*pi} 0 ${0.5*pi}"/>
+                <origin xyz="0 0 0" rpy="0 0 0"/>
                 <geometry>
                     <mesh filename="package://zivid_description/meshes/visual/zivid-one-plus.stl" scale="0.001 0.001 0.001"/>
@@ -26,7 +27,7 @@
             <!-- Collisions -->
             <collision>
-                <origin xyz="-0.0030 -0.0758 0.0445" rpy="${0.5*pi} 0 ${0.5*pi}"/>
+                <origin xyz="0 0 0" rpy="0 0 0"/>
                 <geometry>
-                    <mesh filename="package://zivid_description/meshes/collision/zivid-one-plus.stl" scale="0.001 0.001 0.001"/>
+                    <mesh filename="package://zivid_description/meshes/collision/zivid-one-plus-hull.stl" scale="0.001 0.001 0.001"/>
                 </geometry>
             </collision>
@@ -34,4 +35,6 @@
         <!-- Zivid Optical Frame (Measurement Frame)-->
         <link name="${prefix}optical_frame"/>
+        <!-- Zivid Projector Frame (Projector Optical Frame)-->
+        <link name="${prefix}projector_frame"/>
         <!-- Set the angle of the optical frame based on the type -->
         <xacro:if value="${type == Zivid_One_Plus_S}" >
@@ -50,4 +53,9 @@
             <child link="${prefix}optical_frame"/>
         </joint>
+        <joint name="${prefix}projector_joint" type="fixed">
+            <origin xyz="-0.0030 -0.0758 0.0445" rpy="$0 0 0"/>
+            <parent link="${prefix}base_link"/>
+            <child link="${prefix}projector_frame"/>
+        </joint>
     </xacro:macro>
 </robot>
