Commit message: adjust datums for zivid and bracket

File: urdf/macros/zivid_onarm.xacro (robot description, xacro)
@@ -1,12 +1,8 @@
 <?xml version="1.0"?>
 <robot xmlns:xacro="http://ros.org/wiki/xacro">
-    <!-- Material Properties -->
-    <material name="zivid_gray">
-        <color rgba="0.25 0.25 0.25 1"/>
-    </material>
     <!-- Bracket to put the zivid on a UR arm -->
     <xacro:macro name="zivid_onarm" params="prefix">
         <!-- origin of the mesh is the robot tool flange -->
-        <link name="${prefix}arm_link">
+        <link name="${prefix}base_link">
             <!-- Visuals -->
             <!-- vendor stl was centred on projection frame -->
@@ -32,12 +28,12 @@
         <!-- Zivid mounting joint -->
         <joint name="${prefix}camera_joint" type="fixed">
-            <origin xyz="0 0.065 0.025" rpy="0 -${0.5*pi} -${0.5*pi}"/>
-            <parent link="${prefix}arm_link"/>
+            <origin xyz="0 0.065 0.026" rpy="0 -${0.5*pi} -${0.5*pi}"/>
+            <parent link="${prefix}base_link"/>
             <child link="${prefix}zivid_link"/>
         </joint>
         <!-- gripper joint -->
         <joint name="${prefix}tool_joint" type="fixed">
-            <origin xyz="0 0 12.5" rpy="0 0 0"/>
-            <parent link="${prefix}arm_link"/>
+            <origin xyz="0 0 0.0125" rpy="0 0 0"/>
+            <parent link="${prefix}base_link"/>
             <child link="${prefix}tool_link"/>
         </joint>

File: urdf/macros/zivid_two_camera.xacro (robot description, xacro)
@@ -13,9 +13,5 @@
             <!-- Visuals -->
             <visual>
-                <!-- vendor stl was
-                    rotated by [90,0,90],
-                    translated by -[39.6,84.532,0],
-                    decimated to 3%
-                -->
+                <!-- centered on the 50x50mm bolt pattern -->
                 <origin xyz="0 0 0" rpy="0 0 0"/>
                 <geometry>
@@ -43,5 +39,5 @@
             <!-- Z dimension of optical center is undefined-->
             <origin
-                xyz="0.04702 0.05584 0.0445"
+                xyz="0.02302 0.05584 0.0445"
                 rpy="0 0 ${optical_frame_angle/180*pi}"
             />
@@ -53,6 +49,6 @@
             <!-- projection center is totally undefined-->
             <origin
-                xyz="0.04702 -0.05584 0.0445"
-                rpy="0 0 ${projector_frame_angle)/180*pi}"
+                xyz="0.02302 -0.05584 0.0445"
+                rpy="0 0 ${(projector_frame_angle/180)*pi}"
             />
             <parent link="${prefix}optical_frame"/>
